File: 411_Avionics/Main.sch (EAGLE design)
At the start: 0 parts

Commit message: .... Actually added the .sch file this time.
Parts:
- added C1, C2: 1µ, rcl:C-EU050-025X075
- added CN1: (no value), adafruit:JST_3PIN
- added IC1: BQ24022, texas:BQ24022
- added R1: 4k', rcl:R-US_0309/12
- added U1: (no value), MicroUSB:USB""
Connections:
- new net GND: C1.2, C2.2, CN1.2, IC1G$1.1CE, IC1G$1.ISET2, IC1G$1.VSS, R1.1, U1.GND
- new net N$1: U1.VBUS
- new net N$2: C2.1, IC1G$1.USB
- new net N$3: C1.1, CN1.1, IC1G$1.OUT
- new net N$4: IC1G$1.ISET1, R1.2
Other:
- note added: "Battery Connector"
- note added: "Check Footprint"
