File: eagle/T08-Schematic.sch (EAGLE design)
At the start: 69 parts, among them IC1 BQ24022, J1 USB-MICROB, J3 JST-PH-2-SMT-RA, U1 LP5907, U2 M25P10-AVMN6TP_TR, U3 LSM9DS0, U5 LTC1998, U6 ATMEGA32U4-AU, X1 8MHz

Commit message: Added device for charging chip, and created footprint and device for sensor.
Also began reworking schematic.
Parts:
- removed IC1: BQ24022, tinyav-lib:BQ24022
- removed LED3: (no value), adafruit:LEDCHIP-LED0603
- removed R14: 330, rcl:R-US_R0805
- removed TP18: TPTP08R, testpad:TPTP08R
- added U$1: BQ21040, tinyav-lib:BQ21040
- added U$2: LSM6DS3, tinyav-lib:LSM6DS3
- R1: value 4k -> 5.36k; device rcl:R-US_R0603 -> rcl:R-US_R0805
- R15, R16, R6, R7, R8: value 330 -> 3.3k
Connections:
- removed net N$50: IC1G$1.STAT1, R15.2
- removed net N$51: IC1G$1.STAT2, R14.2
- removed net N$68: IC1G$1./PG, TP18.TP
- net GND: now also U$1.GND; no longer IC1G$1./CE, IC1G$1.ISET2, IC1G$1.VSS
- net N$13: now also U$1.OUT; no longer IC1G$1.OUT
- net N$4: now also R15.2, U$1./CHG; no longer IC1G$1.ISET1, R1.2
- net N$49: now also R1.2, U$1.ISET; no longer LED3.C, R14.1
- net VBUS1: now also U$1.VIN; no longer IC1G$1.USB, LED3.A
Other:
- moved on the sheet: J1, LED2, R1, R15
