File: eagle/tiny-avionics.sch (EAGLE design)
At the start: 62 parts, among them J1 USB-MICROB, J3 JST-PH-2-SMT-RA, U1 LP5907, U2 M25PX16, U3 LSM6DS3, U4 BQ21040, U5 LTC1998, U6 ATMEGA32U4-AU, X1 8MHz

Commit message: Fixed remaining design rev issues. Slightly thinner pads for LSM6DS0 to comply with OshPark DRC.
Connections:
- net N$4: now also U4.!CHG; no longer U4./CHG
Changed lines of the file:
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@@
 <wire x1="71.12" y1="233.68" x2="71.12" y2="236.22" width="0.1524" layer="91"/>
 <wire x1="71.12" y1="236.22" x2="81.28" y2="236.22" width="0.1524" layer="91"/>
-<pinref part="U4" gate="BQ21040" pin="/CHG"/>
+<pinref part="U4" gate="BQ21040" pin="!CHG"/>
 <wire x1="81.28" y1="236.22" x2="81.28" y2="246.38" width="0.1524" layer="91"/>
 </segment>
@@
 </sheet>
 </sheets>
-<errors>
-</errors>
 </schematic>
 </drawing>
